File: ADE7763_Breakout.kicad_sch (KiCad schematic)
At the start: 27 parts, among them J1 10p-2.54, Q1 3.58MHz, U1 ADE7763ARSZSSOP20

Commit message: Fix PCB for footprint and DRC
Parts:
- U1: footprint Package_SO:SSOP-20_4.4x6.5mm_P0.65mm -> Package_SO:SSOP-20_5.3x7.2mm_P0.65mm
Changed lines of the file:
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@@
       (effects (font (size 1.7526 1.7526)) (justify left bottom))
     )
-    (property "Footprint" "Package_SO:SSOP-20_4.4x6.5mm_P0.65mm" (id 2) (at 151.892 99.06 0)
+    (property "Footprint" "Package_SO:SSOP-20_5.3x7.2mm_P0.65mm" (id 2) (at 151.892 99.06 0)
       (effects (font (size 1.27 1.27)) hide)
     )
@@
     )
     (path "/00000000-0000-0000-0000-0000d4dd6c2c"
-      (reference "U1") (unit 1) (value "ADE7763ARSZSSOP20") (footprint "Package_SO:SSOP-20_4.4x6.5mm_P0.65mm")
+      (reference "U1") (unit 1) (value "ADE7763ARSZSSOP20") (footprint "Package_SO:SSOP-20_5.3x7.2mm_P0.65mm")
     )
     (path "/00000000-0000-0000-0000-000040767f2a"
